File: macro1/macro1.kicad_pcb (KiCad board)
At the start: 2 copper layers, 77.5 x 40.6 mm, 8 parts, among them SW1 SW_PUSH, SW2 SW_PUSH, SW4 SW_PUSH, SW5 SW_PUSH, SW6 SW_PUSH, SW7 Rotary_Encoder_Switch, U1 ProMicro_r

Commit message: fix promicro footprint
Routing:
- net GND: track 184.5 -> 182.0 mm
