File: noip/noip.kicad_pcb (KiCad board)
At the start: 2 copper layers, 195.8 x 79.2 mm, 12 parts, among them J2 OLED, SW12 SW_PUSH, SW15 SW_PUSH, SW16 SW_PUSH, SW17 SW_PUSH, SW20 SW_PUSH, SW3 SW_PUSH, SW4 SW_PUSH, SW5 SW_PUSH, SW6 SW_PUSH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

Commit message: oops
Routing:
- net (no net): track 563.0 -> 635.3 mm
Changed lines of the file:
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@@
-(kicad_pcb (version 20171130) (host pcbnew "(5.1.5-0-10_14)")
+(kicad_pcb (version 20171130) (host pcbnew "(5.1.4-0-10_14)")
   (general
     (thickness 1.6)
     (drawings 8)
-    (tracks 71)
+    (tracks 75)
     (zones 0)
     (modules 12)
@@
   (segment (start 150.68 57.902919) (end 150.68 77.7) (width 0.25) (layer F.Cu) (net 0))
   (segment (start 148.14 64.19) (end 148.14 77.7) (width 0.25) (layer F.Cu) (net 0))
+  (segment (start 141.8 92.4) (end 129.8 104.4) (width 0.25) (layer F.Cu) (net 0))
+  (segment (start 141.8 73.09) (end 141.8 92.4) (width 0.25) (layer F.Cu) (net 0))
+  (segment (start 157.015 92.915) (end 168.5 104.4) (width 0.25) (layer F.Cu) (net 0))
+  (segment (start 157.015 73.09) (end 157.015 92.915) (width 0.25) (layer F.Cu) (net 0))
   (segment (start 242 71) (end 232 71) (width 0.25) (layer B.Cu) (net 1))
   (segment (start 222.56316 57.9) (end 214 57.9) (width 0.25) (layer B.Cu) (net 1))
