File: 34Keys/Cradio 10/cradio10.kicad_pcb (KiCad board)
At the start: 2 copper layers, 100.1 x 83.6 mm, 20 parts, among them J1 MJ-4PP-9, SW10 SW_PUSH, SW11 SW_PUSH, SW12 SW_PUSH, SW14 SW_PUSH, SW15 SW_PUSH, SW16 SW_PUSH, SW17 SW_PUSH, SW18 SW_PUSH, SW2 SW_PUSH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

Commit message: Better tidy up, remove duplicates, doh.
Parts:
- moved RSW1 3.06 mm to (130.0, 70.1)
Routing:
- net GND: track 387.5 -> 397.7 mm
- net reset: track 98.1 -> 101.9 mm
