File: 36Keys/besom/besom-r.kicad_pcb (KiCad board)
At the start: 2 copper layers, 109.7 x 81.4 mm, 48 parts, among them J1 MJ-4PP-9, J2 OLED, SW10 SW_PUSH, SW11 SW_PUSH, SW12 SW_PUSH, SW14 SW_PUSH, SW15 SW_PUSH, SW16 SW_PUSH, SW17 SW_PUSH, SW18 SW_PUSH, SW19 SW_PUSH, SW2 SW_PUSH, SW20 SW_PUSH, SW21 SW_PUSH, SW3 SW_PUSH, SW4 SW_PUSH, SW5 SW_PUSH, SW6 SW_PUSH, SW8 SW_PUSH, SW9 SW_PUSH, U1 ProMicro

Commit message: Better tidy up, remove duplicates, doh.
Parts:
- SW14: moved to F.Cu
- U1: footprint kbd:ProMicro_v3 -> kbd:ProMicro_v2
- moved U1 1.25 mm to (135.9, 41.4)
- renumbered JP6 to JP61, JP6 to JP62, JP6 to JP63, JP6 to JP64, JP6 to JP65, JP6 to JP66, JP6 to JP68
Routing:
- net row3: track 108.3 -> 86.7 mm
- net col4: track 126.3 -> 105.3 mm, vias 0 -> 1
- net LED: track 0.00 -> 17.1 mm
- net reset: track 34.3 -> 50.4 mm, vias 2 -> 1
- net SCL: track 32.0 -> 47.9 mm, vias 1 -> 2
- net data: track 43.1 -> 57.9 mm
- net col0: track 0.00 -> 14.4 mm
- net Net-(U1-Pad24): track 0.00 -> 14.4 mm
- net col3: track 111.8 -> 124.3 mm
- net VCC: track 51.0 -> 63.2 mm, vias 1 -> 0
- net col2: track 111.6 -> 122.5 mm, vias 0 -> 1
- net SDA: track 52.6 -> 42.8 mm, vias 1 -> 2
- net row1: track 108.1 -> 102.4 mm, vias 0 -> 1
- net row2: track 108.7 -> 104.4 mm
- net Net-(D14-Pad2): track 14.3 -> 17.4 mm
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Other:
- board size 109.7 x 81.4 mm -> 109.8 x 81.4 mm
