File: 34Keys/hypergolic/hypergolic.kicad_pcb (KiCad board)
At the start: 2 copper layers, 119.4 x 87.6 mm, 28 parts, among them SW10 SW_PUSH, SW11 SW_PUSH, SW12 SW_PUSH, SW14 SW_PUSH, SW15 SW_PUSH, SW16 SW_PUSH, SW17 SW_PUSH, SW18 SW_PUSH, SW2 SW_PUSH, SW20 SW_PUSH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

Commit message: Add files via upload
Parts:
- added REFH1: MountingHole_2.2mm_M2_DIN965_Pad, MountingHole:MountingHole_2.2mm_M2_DIN965_Pad, F.Cu at (109.3, 20.1)
- moved REFH5 19.4 mm to (138.9, 48.0)
Changed lines of the file:
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@@
     (thickness 1.6)
     (drawings 17)
-    (tracks 296)
+    (tracks 298)
     (zones 0)
-    (modules 28)
+    (modules 29)
     (nets 23)
   )
   (page A4)
   (title_block
-    (title "hypergolic")
+    (title hypergolic)
     (date 2020-12-26)
     (rev 0.1)
@@
     (visible_elements FFFFEFFF)
     (pcbplotparams
-      (layerselection 0x010cc_ffffffff)
+      (layerselection 0x010c0_ffffffff)
       (usegerberextensions true)
       (usegerberattributes false)
@@
       (padsonsilk false)
       (subtractmaskfromsilk false)
-      (outputformat 1)
+      (outputformat 3)
       (mirror false)
       (drillshape 0)
       (scaleselection 1)
-      (outputdirectory "gerber/"))
+      (outputdirectory "./"))
   )
   (net 0 "")
@@
   )
   (module MountingHole:MountingHole_2.2mm_M2_DIN965_Pad (layer F.Cu)
-    (at 133.35 66.548)
+    (at 109.256 20.126)
+    (descr "Mounting Hole 2.2mm, M2, DIN965")
+    (tags "mounting hole 2.2mm m2 din965")
+    (attr virtual)
+    (fp_text reference REFH1 (at 0 -2.9) (layer F.SilkS)
+      (effects (font (size 1 1) (thickness 0.15)))
+    )
+    (fp_text value MountingHole_2.2mm_M2_DIN965_Pad (at 0 2.9) (layer F.Fab)
+      (effects (font (size 1 1) (thickness 0.15)))
+    )
+    (fp_circle (center 0 0) (end 1.9 0) (layer Cmts.User) (width 0.15))
+    (fp_circle (center 0 0) (end 2.15 0) (layer F.CrtYd) (width 0.05))
+    (fp_text user %R (at 0.3 0) (layer F.Fab)
+      (effects (font (size 1 1) (thickness 0.15)))
+    )
+    (pad 1 thru_hole circle (at 0 0) (size 3.8 3.8) (drill 2.2) (layers *.Cu *.Mask))
+  )
+  (module MountingHole:MountingHole_2.2mm_M2_DIN965_Pad (layer F.Cu)
+    (at 138.938 48.006)
     (descr "Mounting Hole 2.2mm, M2, DIN965")
     (tags "mounting hole 2.2mm m2 din965")
@@
       (effects (font (size 1 1) (thickness 0.15)))
     )
-    (fp_text user %R (at 0.3 0) (layer F.Fab)
-      (effects (font (size 1 1) (thickness 0.15)))
-    )
     (fp_circle (center 0 0) (end 2.15 0) (layer F.CrtYd) (width 0.05))
     (fp_circle (center 0 0) (end 1.9 0) (layer Cmts.User) (width 0.15))
+    (fp_text user %R (at 0.3 0) (layer F.Fab)
+      (effects (font (size 1 1) (thickness 0.15)))
+    )
     (pad 1 thru_hole circle (at 0 0) (size 3.8 3.8) (drill 2.2) (layers *.Cu *.Mask))
   )
@@
   (gr_line (start 145.288 97.710156) (end 145.288 45.72) (angle 90) (layer Edge.Cuts) (width 0.15))
   (gr_line (start 120.894978 19.479959) (end 89.154 13.462) (angle 90) (layer Edge.Cuts) (width 0.15))
-  (segment (start 130.556 47.244) (end 123.952 40.64) (width 0.25) (layer F.Cu) (net 0))
-  (segment (start 123.952 40.64) (end 123.952 24.638) (width 0.25) (layer F.Cu) (net 0))
-  (segment (start 123.952 24.638) (end 121.92 22.606) (width 0.25) (layer F.Cu) (net 0))
-  (segment (start 97.318 21.238) (end 97.318 20.363) (width 0.25) (layer F.Cu) (net 0))
-  (segment (start 98.686 22.606) (end 97.318 21.238) (width 0.25) (layer F.Cu) (net 0))
-  (segment (start 121.92 22.606) (end 98.686 22.606) (width 0.25) (layer F.Cu) (net 0))
+  (segment (start 123.952 24.638) (end 123.952 40.64) (width 0.25) (layer F.Cu) (net 0))
+  (segment (start 123.063 23.749) (end 123.952 24.638) (width 0.25) (layer F.Cu) (net 0))
+  (segment (start 98.686 22.606) (end 106.426 22.606) (width 0.25) (layer F.Cu) (net 0))
+  (segment (start 123.952 40.64) (end 130.556 47.244) (width 0.25) (layer F.Cu) (net 0))
+  (segment (start 97.318 21.238) (end 98.686 22.606) (width 0.25) (layer F.Cu) (net 0))
+  (segment (start 107.569 23.749) (end 123.063 23.749) (width 0.25) (layer F.Cu) (net 0))
+  (segment (start 106.426 22.606) (end 107.569 23.749) (width 0.25) (layer F.Cu) (net 0))
+  (segment (start 97.318 20.363) (end 97.318 21.238) (width 0.25) (layer F.Cu) (net 0))
   (segment (start 84.58 61.77) (end 86.9162 59.4338) (width 0.25) (layer F.Cu) (net 1))
   (segment (start 86.9162 59.4338) (end 103.9541 59.4338) (width 0.25) (layer F.Cu) (net 1))
